File: Eagle/Radar/radar.sch (EAGLE design)
At the start: 35 parts

Commit message: Added amplifier circuits, ground clips, 3.5mm
Parts:
- added C12: 10uF, rcl:C-EUC0805K
- added C13, C14, C15, C16, C17, C18, C19, C20: (no value), rcl:C-EUC0603
- added IC1, IC2, IC3: AD8519KS, analog-devices:AD8519KS
- added L1: 56 nH, radar:L0603
- added PAD1, PAD2: WIREPADSMD5-2,5, wirepad:WIREPADSMD5-2,5
- added R18, R19, R20, R21, R22, R23, R24, R25, R26, R27, R28, R29: (no value), rcl:R-US_R0603
- added X1: STEREOJACK, adafruit:STEREOJACK
- C11: value 10uF -> (none); device rcl:C-EUC0805K -> rcl:C-EUC0603; DIGI 587-2985-1-ND -> (none)
- R17: value 0 -> 191, 1/2W; device rcl:R-US_R0201 -> rcl:R-US_R1210; DIGI (none) -> P191AACT-ND
Connections:
- new net N$1: C20.1, R25.2
- new net N$10: IC3.OUT, R19.1, R24.2
- new net N$11: IC3.IN-, R24.1, R28.2
- new net N$12: C19.2, IC3.IN+, R29.2
- new net N$13: C19.1
- new net N$14: C20.2, X1.2
- new net N$2: C11.2, R18.1, R19.2
- new net N$3: C11.1, C15.1, IC1.OUT, IC2.OUT, R20.1, R21.2, R25.1, R26.2
- new net N$6: C13.1, C16.1, IC1.IN+, IC2.IN+, R18.2, R23.2
- new net N$7: C14.1, C17.1, C18.1, IC1.+VS, IC2.+VS
- new net N$8: IC1.IN-, IC2.IN-, R21.1, R22.2, R26.1, R27.2
- new net N$9: C15.2, R20.2, R23.1
- net AMP_OUT: now also L1.2
- net AMP_VCC: now also L1.1; no longer C11.1
- net GND: now also C12.2, C13.2, C14.2, C16.2, C17.2, C18.2, IC1.-VS, IC2.-VS, IC3.-VS, PAD1.P, PAD2.P, R22.1, R27.1, R28.1, R29.1, X1.1; no longer C11.2
- net PP10V: now also C12.1
Other:
- note added: "Ground clips"
- moved on the sheet: C11, R17

Commit message: Updated schematic
Parts:
- removed IC1, IC2, IC3: AD8519KS, analog-devices:AD8519KS
- added C21, C22: 10uF, rcl:C-EUC0805K
- added C23: 0.1u, rcl:C-EUC0603
- added IC4: MAX414ESD, radar:MAX414ESD
- added JP1: (no value), pinhead:PINHD-1X2
- added R30: 0, rcl:R-US_R0402
- added R31: 50, rcl:R-US_R0603
- added U$10: DMN3067LW-7, radar:DMN3067LW-7
- added U$9: COUPLER, radar:COUPLER
- added X2, X3, X4: BU-SMA-G, radar:BU-SMA-G
- C14, C19: value (none) -> 10uF; device rcl:C-EUC0603 -> rcl:C-EUC0805K; DIGI (none) -> 587-2985-1-ND
- C17: value (none) -> 270p; device rcl:C-EUC0603 -> rcl:C-EUC0603K; DIGI (none) -> 399-9054-1-ND
- C18: value (none) -> 0.1u; DIGI (none) -> 311-1088-1-ND
- R2, R5, R8: device rcl:R-US_R0201 -> rcl:R-US_R0402
- U$7: value CVCO55CC-2380-2580 -> MAX268X; device radar:CVCO55CC-2380-2580 -> radar:MAX268X
Connections:
- net N$1 renamed AUD1_AC
- net N$14 renamed AUD1_OUT
- net N$2 renamed LFA2_IN
- net N$9 renamed LFA3_IN
- removed net N$10: IC3.OUT, R19.1, R24.2
- removed net N$11: IC3.IN-, R24.1, R28.2
- removed net N$12: C19.2, IC3.IN+, R29.2
- removed net N$13: C19.1
- removed net N$3: C11.1, C15.1, IC1.OUT, IC2.OUT, R20.1, R21.2, R25.1, R26.2
- removed net N$4: C9.2
- removed net N$5: C10.1
- removed net N$6: C13.1, C16.1, IC1.IN+, IC2.IN+, R18.2, R23.2
- removed net N$7: C14.1, C17.1, C18.1, IC1.+VS, IC2.+VS
- removed net N$8: IC1.IN-, IC2.IN-, R21.1, R22.2, R26.1, R27.2
- removed net VCO_RF: U$7.RF_OUT
- removed net VCO_VT: U$7.VT
- new net COUPLER_COUPLED: C14.2, U$9.COUPLED
- new net COUPLER_IN: C10.1, U$9.RF_IN
- new net COUPLER_ISO: R31.2, U$9.ISOLATE
- new net COUPLER_OUT: U$9.THRU, X4.1
- new net LFA1_+: C19.1, IC4A.+IN, R29.2
- new net LFA1_-: IC4A.-IN, R24.1, R28.2
- new net LFA1_OUT: IC4A.OUT, R19.1, R24.2
- new net LFA2_+: C13.1, IC4B.+IN, R18.2
- new net LFA2_-: IC4B.-IN, R21.1, R22.2
- new net LFA2_OUT: C11.1, IC4B.OUT, R20.1, R21.2
- new net LFA3_+: C16.1, IC4C.+IN, R23.2
- new net LFA3_-: IC4C.-IN, R26.1, R27.2
- new net LFA3_OUT: C15.1, IC4C.OUT, R25.1, R26.2
- new net MAX268X_SHDN: R30.1, U$7.SHDN_N
- new net MIXER_IF: C19.2, U$7.IF
- new net MIXER_LO: C14.1, U$7.LO
- new net MIXER_RF: C17.1, U$7.RF
- new net MOTOR_CTRL: U$10.G, U$3.D6
- new net N$1: JP1.2, U$10.D
- new net PLL_OUT: C9.2, X2.1
- new net RF_RX: C17.2, X3.1
- net GND: now also C21.2, C22.2, C23.2, IC4A.V-, R31.1, U$10.S, U$7.GND, X2.2, X3.2, X4.2; no longer C14.2, C17.2, IC1.-VS, IC2.-VS, IC3.-VS, U$7.GND@1, U$7.GND@11, U$7.GND@12, U$7.GND@13, U$7.GND@15, U$7.GND@16, U$7.GND@3, U$7.GND@4, U$7.GND@5, U$7.GND@6, U$7.GND@7, U$7.GND@8, U$7.GND@9
- net PP10V: now also C18.1, C22.1, IC4A.V+
- net PP5V: now also C21.1, C23.1, R30.2
- net PPUSB: now also JP1.1
Other:
- moved on the sheet: C1, C10, C11, C12, C13, C14, C15, C16, C17, C18, C19, C2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

Commit message: Updated digi values
Parts:
- removed C7, C8: 10uF, rcl:C-EUC0805K
- removed R10: 4.48k, rcl:R-US_R0603
- removed R15, R16: 0, rcl:R-US_R0603
- removed R9: 2.61k, rcl:R-US_R0603
- removed U$6: TPS73801, radar:TPS73801
- added L2: 1.2nH, radar:L0603
- added R32: 28k, rcl:R-US_R0603
- C11, C13, C15, C16: value (none) -> 1n; DIGI (none) -> 311-1085-1-ND
- C20: value (none) -> 10uF; device rcl:C-EUC0603 -> rcl:C-EUC0805K; DIGI (none) -> 587-2985-1-ND
- R18: value (none) -> 7.15k; DIGI (none) -> 311-7.15KHRCT-ND
- R19: value (none) -> 8.25k; DIGI (none) -> RNCP0805FTD8K25CT-ND
- R20: value (none) -> 17.4k; DIGI (none) -> 311-17.4KHRCT-ND
- R21, R26: value (none) -> 1k; DIGI (none) -> 311-1.00KHRCT-ND
- R22: value (none) -> 12.1k; DIGI (none) -> 541-12.1KSCT-ND
- R23: value (none) -> 4.12k; DIGI (none) -> 311-4.12KHRCT-ND
- R24: value (none) -> 100k; DIGI (none) -> 541-3247-1-ND
- R25: value (none) -> 0
- R27: value (none) -> 1.2k; DIGI (none) -> 311-1.20KHRCT-ND
- R28: value (none) -> 200; DIGI (none) -> RNCP0805FTD200RCT-ND
- R29: value (none) -> 10k; DIGI (none) -> 311-10.0KHRCT-ND
- R31: DIGI (none) -> RNCP0805FTD49R9CT-ND
- R8: value 0 -> 20k; device rcl:R-US_R0402 -> pot:TRIM_US-B25P; DIGI (none) -> 3362P-203LF-ND
- U$7: DIGI (none) -> MAX2682EUT+TCT-ND
Connections:
- removed net LDO3_EN: R8.2, U$6.EN
- removed net LDO3_FB: R10.1, R9.2, U$6.FB
- removed net LDO3_IN: C7.1, R15.2, R8.1, U$6.IN
- removed net LDO3_OUT: C8.1, R10.2, R16.1, U$6.OUT
- removed net PP3V3: R16.2
- net GND: now also L2.2; no longer C13.2, C16.2, C7.2, C8.2, R22.1, R27.1, R28.1, R29.1, R9.1, U$6.GND@1, U$6.GND@2
- net LFA1_-: now also R8.A, R8.S; no longer R24.1
- net LFA1_OUT: now also R8.E; no longer R24.2
- net LFA2_IN: now also R24.2
- net LFA3_IN: now also R32.2
- net PP5V: now also C13.2, C16.2, R22.1, R24.1, R27.1, R28.1, R29.1, R32.1; no longer R15.1
- net RF_RX: now also L2.1
Other:
- note removed: "Vout=3.300V"
- moved on the sheet: C11, C15, JP1, R24, R28, U$10, X3

Commit message: Finalized sch
Parts:
- added C7: 10uF, rcl:C-EUC0805K
- added JP2: (no value), pinhead:PINHD-1X4
- added JP3: (no value), pinhead:PINHD-1X2
- added L3: 56 nH, radar:L0603
- added U$6: COUPLER, radar:COUPLER
- L2: DIGI 712-1443-1-ND -> 535-11530-1-ND
- U$9: value COUPLER -> PAT1220; device radar:COUPLER -> radar:PAT1220; DIGI (none) -> PAT123CT-ND
Connections:
- new net AUD2_OUT: C7.2, X1.5
- new net AUD2_PLACEHOLDER: C7.1
- new net ENCODER_A: JP2.2
- new net ENCODER_B: JP2.3, U$3.D2
- new net N$2: C9.2, U$9.RF_OUT
- net COUPLER_COUPLED: now also U$6.COUPLED; no longer U$9.COUPLED
- net COUPLER_IN: now also U$6.RF_IN; no longer U$9.RF_IN
- net COUPLER_ISO: now also U$6.ISOLATE; no longer U$9.ISOLATE
- net COUPLER_OUT: now also U$6.THRU; no longer U$9.THRU
- net GND: now also JP2.4, JP3.2, U$9.GND
- net MIXER_IF: now also L3.2
- net PLL_OUT: now also U$9.RF_IN; no longer C9.2
- net PP5V: now also JP2.1, L3.1
- net PPUSB: now also JP3.1
Other:
- moved on the sheet: C1, C2, C3, C4, C5, C6, JP1, PAD1, PAD2, R1, R11, R12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

Commit message: Nearly completed placements on board
Parts:
- removed R11, R12, R13, R14, R25: 0, rcl:R-US_R0603
- removed R30, R5: 0, rcl:R-US_R0402
- added C24, C25, C8: 10uF, rcl:C-EUC0805K
- added L4: 56 nH, radar:L0603
- added SJ1, SJ2, SJ3, SJ4, SJ5, SJ6, SJ7, SJ8, SJ9: (no value), jumper:SJ
- added U$11: ERA3+, radar:ERA3+
- R2: value 0 -> 191, 1/2W; device rcl:R-US_R0402 -> rcl:R-US_R1210; DIGI (none) -> P191AACT-ND
Connections:
- net N$2 renamed ATTEN_OUT
- net PLL_OUT renamed PLL_IN
- new net LNA_IN: C8.1, U$11.RF_IN
- new net LNA_OUT: C24.2, L4.2, U$11.RF_OUT
- new net LNA_VCC: L4.1, R2.1
- new net MOTOR_GATE: SJ9.2, U$10.G
- new net N$3: C8.2, X3.1
- net AUD1_AC: now also SJ2.2; no longer R25.2
- net GND: now also C25.2, U$11.GND@2, U$11.GND@4
- net LDO1_EN: now also SJ5.2; no longer R2.2
- net LDO1_IN: now also SJ5.1, SJ6.2; no longer R12.2, R2.1
- net LDO1_OUT: now also SJ4.1; no longer R13.1
- net LDO2_EN: now also SJ8.2; no longer R5.2
- net LDO2_IN: now also SJ7.2, SJ8.1; no longer R11.2, R5.1
- net LDO2_OUT: now also SJ3.1; no longer R14.1
- net LFA2_+: now also IC4D.+IN; no longer IC4B.+IN
- net LFA2_-: now also IC4D.-IN; no longer IC4B.-IN
- net LFA2_OUT: now also IC4D.OUT; no longer IC4B.OUT
- net LFA3_OUT: now also SJ2.1; no longer R25.1
- net MAX268X_SHDN: now also SJ1.1; no longer R30.1
- net MOTOR_CTRL: now also SJ9.1; no longer U$10.G
- net PP10V: now also C25.1, R2.2, SJ4.2, SJ7.1; no longer R11.1, R13.2
- net PP10V4: now also SJ6.1; no longer R12.1
- net PP5V: now also SJ1.2, SJ3.2; no longer R14.2, R30.2
- net RF_RX: now also C24.1; no longer X3.1
Other:
- moved on the sheet: C9, IC4D, R2, U$9, X3

Commit message: Routing complete
Parts:
- removed SJ5, SJ8: (no value), jumper:SJ
- added C26, C27, C28: 0.1u, rcl:C-EUC0603
- added JP4: (no value), pinhead:PINHD-1X2
Connections:
- removed net LDO1_EN: SJ5.2, U$1.EN
- removed net LDO2_EN: SJ8.2, U$5.EN
- net ENCODER_A: now also U$3.D2
- net ENCODER_B: now also U$3.D3; no longer U$3.D2
- net GND: now also C26.2, C27.2, C28.2, JP4.2
- net LDO1_IN: now also U$1.EN; no longer SJ5.1
- net LDO2_IN: now also U$5.EN; no longer SJ8.1
- net PP10V: now also JP4.1
- net PP5V: now also C26.1, C27.1, C28.1
Other:
- note added: "EXT Power conn"
- note added: "Encoder conn"
- note added: "Motor conn"
- note added: "PLL Power conn"
Changed lines of the file:
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@@
 <part name="SJ3" library="jumper" deviceset="SJ" device=""/>
 <part name="SJ4" library="jumper" deviceset="SJ" device=""/>
-<part name="SJ5" library="jumper" deviceset="SJ" device=""/>
 <part name="SJ6" library="jumper" deviceset="SJ" device=""/>
 <part name="SJ7" library="jumper" deviceset="SJ" device=""/>
-<part name="SJ8" library="jumper" deviceset="SJ" device=""/>
 <part name="SJ9" library="jumper" deviceset="SJ" device=""/>
 <part name="C8" library="rcl" deviceset="C-EU" device="C0805K" value="10uF">
@@
 </part>
 <part name="SUPPLY21" library="supply2" deviceset="GND" device=""/>
+<part name="C26" library="rcl" deviceset="C-EU" device="C0603" value="0.1u">
+<attribute name="DIGI" value="311-1088-1-ND"/>
+</part>
+<part name="C27" library="rcl" deviceset="C-EU" device="C0603" value="0.1u">
+<attribute name="DIGI" value="311-1088-1-ND"/>
+</part>
+<part name="C28" library="rcl" deviceset="C-EU" device="C0603" value="0.1u">
+<attribute name="DIGI" value="311-1088-1-ND"/>
+</part>
+<part name="SUPPLY26" library="supply2" deviceset="GND" device=""/>
+<part name="SUPPLY29" library="supply2" deviceset="GND" device=""/>
+<part name="SUPPLY30" library="supply2" deviceset="GND" device=""/>
+<part name="JP4" library="pinhead" deviceset="PINHD-1X2" device=""/>
+<part name="SUPPLY33" library="supply2" deviceset="GND" device=""/>
 </parts>
 <sheets>
@@
 <text x="360.68" y="208.28" size="1.778" layer="97">Vout=5.036V</text>
 <text x="63.5" y="266.7" size="1.778" layer="97">Ground clips</text>
+<text x="139.7" y="185.42" size="1.778" layer="97" rot="R90">Encoder conn</text>
+<text x="208.28" y="198.12" size="1.778" layer="97" rot="R90">Motor conn</text>
+<text x="139.7" y="157.48" size="1.778" layer="97" rot="R90">EXT Power conn</text>
+<text x="180.34" y="157.48" size="1.778" layer="97" rot="R90">PLL Power conn</text>
 </plain>
 <instances>
@@
 <instance part="SJ3" gate="1" x="406.4" y="205.74"/>
 <instance part="SJ4" gate="1" x="406.4" y="254"/>
-<instance part="SJ5" gate="1" x="304.8" y="248.92"/>
 <instance part="SJ6" gate="1" x="266.7" y="254"/>
 <instance part="SJ7" gate="1" x="266.7" y="205.74"/>
-<instance part="SJ8" gate="1" x="304.8" y="200.66"/>
 <instance part="SJ9" gate="1" x="187.96" y="187.96"/>
 <instance part="C8" gate="G$1" x="-60.96" y="68.58" rot="R270">
@@
 <instance part="SUPPLY21" gate="GND" x="35.56" y="76.2"/>
 <instance part="IC4" gate="D" x="297.18" y="63.5"/>
+<instance part="C26" gate="G$1" x="215.9" y="22.86">
+<attribute name="DIGI" x="215.9" y="22.86" size="1.778" layer="96" display="off"/>
+</instance>
+<instance part="C27" gate="G$1" x="264.16" y="38.1">
+<attribute name="DIGI" x="264.16" y="38.1" size="1.778" layer="96" display="off"/>
+</instance>
+<instance part="C28" gate="G$1" x="314.96" y="25.4">
+<attribute name="DIGI" x="314.96" y="25.4" size="1.778" layer="96" display="off"/>
+</instance>
+<instance part="SUPPLY26" gate="GND" x="215.9" y="12.7"/>
+<instance part="SUPPLY29" gate="GND" x="264.16" y="27.94"/>
+<instance part="SUPPLY30" gate="GND" x="314.96" y="15.24"/>
+<instance part="JP4" gate="G$1" x="187.96" y="170.18"/>
+<instance part="SUPPLY33" gate="GND" x="193.04" y="165.1"/>
 </instances>
 <busses>
@@
 <pinref part="SUPPLY21" gate="GND" pin="GND"/>
 <wire x1="35.56" y1="78.74" x2="35.56" y2="81.28" width="0.1524" layer="91"/>
+</segment>
+<segment>
+<pinref part="C26" gate="G$1" pin="2"/>
+<pinref part="SUPPLY26" gate="GND" pin="GND"/>
+<wire x1="215.9" y1="15.24" x2="215.9" y2="17.78" width="0.1524" layer="91"/>
+</segment>
+<segment>
+<pinref part="C27" gate="G$1" pin="2"/>
+<pinref part="SUPPLY29" gate="GND" pin="GND"/>
+<wire x1="264.16" y1="30.48" x2="264.16" y2="33.02" width="0.1524" layer="91"/>
+</segment>
+<segment>
+<pinref part="C28" gate="G$1" pin="2"/>
+<pinref part="SUPPLY30" gate="GND" pin="GND"/>
+<wire x1="314.96" y1="17.78" x2="314.96" y2="20.32" width="0.1524" layer="91"/>
+</segment>
+<segment>
+<pinref part="JP4" gate="G$1" pin="2"/>
+<wire x1="185.42" y1="170.18" x2="193.04" y2="170.18" width="0.1524" layer="91"/>
+<pinref part="SUPPLY33" gate="GND" pin="GND"/>
+<wire x1="193.04" y1="167.64" x2="193.04" y2="170.18" width="0.1524" layer="91"/>
 </segment>
 </net>
@@
 <pinref part="R28" gate="G$1" pin="1"/>
 <wire x1="226.06" y1="27.94" x2="226.06" y2="30.48" width="0.1524" layer="91"/>
-<wire x1="226.06" y1="27.94" x2="208.28" y2="27.94" width="0.1524" layer="91"/>
+<wire x1="226.06" y1="27.94" x2="215.9" y2="27.94" width="0.1524" layer="91"/>
 <label x="208.28" y="27.94" size="1.778" layer="95"/>
+<pinref part="C26" gate="G$1" pin="1"/>
+<wire x1="215.9" y1="27.94" x2="208.28" y2="27.94" width="0.1524" layer="91"/>
+<wire x1="215.9" y1="25.4" x2="215.9" y2="27.94" width="0.1524" layer="91"/>
+<junction x="215.9" y="27.94"/>
 </segment>
 <segment>
@@
 <junction x="256.54" y="48.26"/>
 <wire x1="256.54" y1="48.26" x2="256.54" y2="43.18" width="0.1524" layer="91"/>
-<wire x1="256.54" y1="43.18" x2="266.7" y2="43.18" width="0.1524" layer="91"/>
+<wire x1="256.54" y1="43.18" x2="264.16" y2="43.18" width="0.1524" layer="91"/>
 <label x="259.08" y="43.18" size="1.778" layer="95"/>
+<pinref part="C27" gate="G$1" pin="1"/>
+<wire x1="264.16" y1="43.18" x2="266.7" y2="43.18" width="0.1524" layer="91"/>
+<wire x1="264.16" y1="40.64" x2="264.16" y2="43.18" width="0.1524" layer="91"/>
+<junction x="264.16" y="43.18"/>
 </segment>
 <segment>
 <pinref part="R22" gate="G$1" pin="1"/>
 <wire x1="325.12" y1="30.48" x2="325.12" y2="33.02" width="0.1524" layer="91"/>
-<wire x1="325.12" y1="30.48" x2="312.42" y2="30.48" width="0.1524" layer="91"/>
+<wire x1="325.12" y1="30.48" x2="314.96" y2="30.48" width="0.1524" layer="91"/>
 <label x="312.42" y="30.48" size="1.778" layer="95"/>
+<pinref part="C28" gate="G$1" pin="1"/>
+<wire x1="314.96" y1="30.48" x2="312.42" y2="30.48" width="0.1524" layer="91"/>
+<wire x1="314.96" y1="27.94" x2="314.96" y2="30.48" width="0.1524" layer="91"/>
+<junction x="314.96" y="30.48"/>
 </segment>
 <segment>
@@
 <label x="152.4" y="198.12" size="1.778" layer="95"/>
 <pinref part="JP2" gate="A" pin="1"/>
-</segment>
-</net>
-<net name="LDO1_EN" class="0">
-<segment>
-<pinref part="U$1" gate="G$1" pin="EN"/>
-<wire x1="309.88" y1="248.92" x2="325.12" y2="248.92" width="0.1524" layer="91"/>
-<label x="312.42" y="248.92" size="1.778" layer="95"/>
-<pinref part="SJ5" gate="1" pin="2"/>
 </segment>
 </net>
@@
 <junction x="35.56" y="91.44"/>
 </segment>
-</net>
-<net name="LDO2_EN" class="0">
-<segment>
-<pinref part="U$5" gate="G$1" pin="EN"/>
-<wire x1="309.88" y1="200.66" x2="325.12" y2="200.66" width="0.1524" layer="91"/>
-<label x="312.42" y="200.66" size="1.778" layer="95"/>
-<pinref part="SJ8" gate="1" pin="2"/>
+<segment>
+<pinref part="JP4" gate="G$1" pin="1"/>
+<wire x1="185.42" y1="172.72" x2="208.28" y2="172.72" width="0.1524" layer="91"/>
+<label x="193.04" y="172.72" size="1.778" layer="95"/>
 </segment>
 </net>
@@
 <wire x1="287.02" y1="254" x2="287.02" y2="251.46" width="0.1524" layer="91"/>
 <junction x="287.02" y="254"/>
-<wire x1="299.72" y1="248.92" x2="297.18" y2="248.92" width="0.1524" layer="91"/>
 <wire x1="297.18" y1="248.92" x2="297.18" y2="254" width="0.1524" layer="91"/>
 <junction x="297.18" y="254"/>
 <label x="274.32" y="254" size="1.778" layer="95"/>
 <wire x1="271.78" y1="254" x2="287.02" y2="254" width="0.1524" layer="91"/>
-<pinref part="SJ5" gate="1" pin="1"/>
 <pinref part="SJ6" gate="1" pin="2"/>
+<pinref part="U$1" gate="G$1" pin="EN"/>
+<wire x1="297.18" y1="248.92" x2="325.12" y2="248.92" width="0.1524" layer="91"/>
+<label x="312.42" y="248.92" size="1.778" layer="95"/>
 </segment>
 </net>
@@
 <pinref part="U$5" gate="G$1" pin="IN"/>
 <wire x1="325.12" y1="205.74" x2="297.18" y2="205.74" width="0.1524" layer="91"/>
-<wire x1="299.72" y1="200.66" x2="297.18" y2="200.66" width="0.1524" layer="91"/>
 <wire x1="297.18" y1="200.66" x2="297.18" y2="205.74" width="0.1524" layer="91"/>
 <junction x="297.18" y="205.74"/>
@@
 <label x="274.32" y="205.74" size="1.778" layer="95"/>
 <pinref part="SJ7" gate="1" pin="2"/>
-<pinref part="SJ8" gate="1" pin="1"/>
+<pinref part="U$5" gate="G$1" pin="EN"/>
+<wire x1="297.18" y1="200.66" x2="325.12" y2="200.66" width="0.1524" layer="91"/>
+<label x="312.42" y="200.66" size="1.778" layer="95"/>
 </segment>
 </net>
@@
 </segment>
 <segment>
+<wire x1="154.94" y1="238.76" x2="172.72" y2="238.76" width="0.1524" layer="91"/>
+<label x="157.48" y="238.76" size="1.778" layer="95"/>
+<pinref part="U$3" gate="G$1" pin="D3"/>
+</segment>
+</net>
+<net name="ENCODER_A" class="0">
+<segment>
+<wire x1="144.78" y1="195.58" x2="167.64" y2="195.58" width="0.1524" layer="91"/>
+<label x="152.4" y="195.58" size="1.778" layer="95"/>
+<pinref part="JP2" gate="A" pin="2"/>
+</segment>
+<segment>
 <pinref part="U$3" gate="G$1" pin="D2"/>
 <wire x1="154.94" y1="236.22" x2="172.72" y2="236.22" width="0.1524" layer="91"/>
@@
 </segment>
 </net>
-<net name="ENCODER_A" class="0">
-<segment>
-<wire x1="144.78" y1="195.58" x2="167.64" y2="195.58" width="0.1524" layer="91"/>
-<label x="152.4" y="195.58" size="1.778" layer="95"/>
-<pinref part="JP2" gate="A" pin="2"/>
-</segment>
-<segment>
-<wire x1="154.94" y1="238.76" x2="172.72" y2="238.76" width="0.1524" layer="91"/>
-<label x="157.48" y="238.76" size="1.778" layer="95"/>
-</segment>
-</net>
