File: Eagle/Radar/radar.sch (EAGLE design)
At the start: 86 parts, among them IC4 MAX414ESD, X1 STEREOJACK, X2 BU-SMA-G, X3 BU-SMA-G, X4 BU-SMA-G

Commit message: Design complete
Connections:
- net N$3 renamed RF__RX_IN
Other:
- moved on the sheet: X3
Changed lines of the file:
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@@
 <attribute name="DIGI" x="33.02" y="68.58" size="1.778" layer="96" rot="R270" display="off"/>
 </instance>
-<instance part="SUPPLY31" gate="GND" x="-71.12" y="55.88"/>
+<instance part="SUPPLY31" gate="GND" x="-78.74" y="55.88"/>
 <instance part="C19" gate="G$1" x="172.72" y="68.58" rot="R270">
 <attribute name="DIGI" x="172.72" y="68.58" size="1.778" layer="96" rot="R270" display="off"/>
@@
 <attribute name="DIGI" x="129.54" y="137.16" size="1.778" layer="96" display="off"/>
 </instance>
-<instance part="X3" gate="G1" x="-78.74" y="68.58">
-<attribute name="DIGI" x="-78.74" y="68.58" size="1.778" layer="96" display="off"/>
+<instance part="X3" gate="G1" x="-86.36" y="68.58">
+<attribute name="DIGI" x="-86.36" y="68.58" size="1.778" layer="96" display="off"/>
 </instance>
 <instance part="X4" gate="G1" x="383.54" y="137.16" rot="MR0">
@@
 </segment>
 <segment>
-<wire x1="-76.2" y1="66.04" x2="-71.12" y2="66.04" width="0.1524" layer="91"/>
+<wire x1="-83.82" y1="66.04" x2="-78.74" y2="66.04" width="0.1524" layer="91"/>
 <pinref part="SUPPLY31" gate="GND" pin="GND"/>
-<wire x1="-71.12" y1="66.04" x2="-71.12" y2="58.42" width="0.1524" layer="91"/>
+<wire x1="-78.74" y1="66.04" x2="-78.74" y2="58.42" width="0.1524" layer="91"/>
 <pinref part="X3" gate="G1" pin="2"/>
 </segment>
@@
 <pinref part="C17" gate="G$1" pin="2"/>
 <wire x1="27.94" y1="68.58" x2="22.86" y2="68.58" width="0.1524" layer="91"/>
-<label x="-73.66" y="68.58" size="1.778" layer="95"/>
 <pinref part="L2" gate="G$1" pin="1"/>
 <wire x1="22.86" y1="66.04" x2="22.86" y2="68.58" width="0.1524" layer="91"/>
@@
 </segment>
 </net>
-<net name="N$3" class="0">
+<net name="RF__RX_IN" class="0">
 <segment>
 <pinref part="C8" gate="G$1" pin="2"/>
-<wire x1="-66.04" y1="68.58" x2="-76.2" y2="68.58" width="0.1524" layer="91"/>
+<wire x1="-66.04" y1="68.58" x2="-83.82" y2="68.58" width="0.1524" layer="91"/>
 <pinref part="X3" gate="G1" pin="1"/>
-</segment>
-</net>
+<label x="-81.28" y="68.58" size="1.778" layer="95"/>
+</segment>
+</net>
